File: IdealDiode.kicad_sch (KiCad schematic)
At the start: 0 parts

Commit message: Designed PCB, parallelized it, ready for submission
Parts:
- added D1, D2: PMEG2020EH, Diode_SMD:D_SOD-123F, symbol Diode:PMEG2020EH
- added J1, J2, J3, J4: Conn_01x01_Pin, Connector_PinSocket_2.54mm:PinSocket_1x01_P2.54mm_Vertical, symbol Connector:Conn_01x01_Pin
- added Q1: AO3400A, Package_TO_SOT_SMD:SOT-23, symbol Transistor_FET:AO3400A
- added Q2: AO3401A, Package_TO_SOT_SMD:SOT-23, symbol Transistor_FET:AO3401A
- added R1, R2: 10k, Resistor_SMD:R_0402_1005Metric, symbol Device:R_Small
- added U1: LM393, Package_SO:VSSOP-8_3x3mm_P0.65mm, symbol Comparator:LM393
Connections:
- new net: Q1.3 (D), Q2.1 (G), R1.1
- new net: Q1.1 (G), R2.2, U1.1
- new net GND: J2.1 (Pin_1), J4.1 (Pin_1), Q1.2 (S), U1.4 (V-)
- new net a: D1.1 (K), D2.1 (K), R1.2, R2.1, U1.8 (V+)
- new net i: D1.2 (A), J1.1 (Pin_1), Q2.3 (D), U1.3 (+)
- new net o: D2.2 (A), J3.1 (Pin_1), Q2.2 (S), U1.2 (-)
