File: Panelize.kicad_pcb (KiCad board)
At the start: 2 copper layers, 13.7 x 18.3 mm, 22 parts, among them J1 Conn_01x01_Pin, J2 Conn_01x01_Pin, J3 Conn_01x01_Pin, J4 Conn_01x01_Pin, Q1 AO3400A, Q2 AO3401A, U1 LM393

Commit message: Adjusted design for panel production
Other:
- board size 13.7 x 18.3 mm -> 17.8 x 22.9 mm
- board text removed: "V-CUT"
