File: IdealDiode/IdealDiode.kicad_pcb (KiCad board)
At the start: 2 copper layers, 13.7 x 9.1 mm, 11 parts, among them J1 Conn_01x01_Pin, J2 Conn_01x01_Pin, J3 Conn_01x01_Pin, J4 Conn_01x01_Pin, Q1 AO3400A, Q2 AO3401A, U1 LM393

Commit message: Moved PCB files to respective folders, adjusted netlabels
Connections:
- net /a renamed /anydir
- net /i renamed /in
- net /o renamed /out
