File: IdealDiode/IdealDiode.kicad_sch (KiCad schematic)
At the start: 11 parts, among them J1 Conn_01x01_Pin, J2 Conn_01x01_Pin, J3 Conn_01x01_Pin, J4 Conn_01x01_Pin, Q1 AO3400A, Q2 AO3401A, U1 LM393

Commit message: Moved PCB files to respective folders, adjusted netlabels
Connections:
- net a renamed anydir
- net i renamed in
- net o renamed out
Changed lines of the file:
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@@
+	(wire
+		(pts
+			(xy 77.47 133.35) (xy 81.28 133.35)
+		)
+		(stroke
+			(width 0)
+			(type default)
+		)
+	)
 	(wire
 		(pts
@@
 	(wire
 		(pts
-			(xy 81.28 137.16) (xy 81.28 133.35)
+			(xy 77.47 135.89) (xy 77.47 133.35)
 		)
 		(stroke
@@
 		)
 	)
-	(label "o"
+	(label "in"
+		(at 83.82 162.56 0)
+		(effects
+			(font
+				(size 1.27 1.27)
+			)
+			(justify left bottom)
+		)
+	)
+	(label "out"
 		(at 62.23 111.76 180)
 		(effects
@@
 		)
 	)
-	(label "o"
+	(label "out"
+		(at 88.9 160.02 180)
+		(effects
+			(font
+				(size 1.27 1.27)
+			)
+			(justify right bottom)
+		)
+	)
+	(label "anydir"
+		(at 104.14 132.08 180)
+		(effects
+			(font
+				(size 1.27 1.27)
+			)
+			(justify right bottom)
+		)
+	)
+	(label "in"
+		(at 54.61 111.76 0)
+		(effects
+			(font
+				(size 1.27 1.27)
+			)
+			(justify left bottom)
+		)
+	)
+	(label "in"
+		(at 77.47 123.19 0)
+		(effects
+			(font
+				(size 1.27 1.27)
+			)
+			(justify left bottom)
+		)
+	)
+	(label "out"
 		(at 107.95 123.19 180)
 		(effects
@@
 		)
 	)
-	(label "a"
-		(at 104.14 132.08 180)
-		(effects
-			(font
-				(size 1.27 1.27)
-			)
-			(justify right bottom)
-		)
-	)
-	(label "i"
-		(at 83.82 162.56 0)
-		(effects
-			(font
-				(size 1.27 1.27)
-			)
-			(justify left bottom)
-		)
-	)
-	(label "i"
-		(at 54.61 111.76 0)
-		(effects
-			(font
-				(size 1.27 1.27)
-			)
-			(justify left bottom)
-		)
-	)
-	(label "i"
-		(at 77.47 123.19 0)
-		(effects
-			(font
-				(size 1.27 1.27)
-			)
-			(justify left bottom)
-		)
-	)
-	(label "a"
+	(label "anydir"
 		(at 53.34 130.81 180)
 		(effects
@@
 		)
 	)
-	(label "o"
-		(at 88.9 160.02 180)
-		(effects
-			(font
-				(size 1.27 1.27)
-			)
-			(justify right bottom)
-		)
-	)
-	(label "a"
-		(at 81.28 137.16 0)
-		(effects
-			(font
+	(label "anydir"
+		(at 77.47 135.89 0)
+		(effects
+			(font
